Commit message: feat: add IMU sensor to robot description and update Rviz configuration for new robot link names and navigation planner topics.

File: src/sme_robot_mobile_description/urdf/sme_robot_mobile_sensors.xacro (robot description, xacro)
@@ -77,4 +77,50 @@
       </sensor>
     </gazebo>
+    <!--
+      IMU SENSOR
+      Used for orientation and acceleration measurements.
+    -->
+    <link name="${name}_imu_link">
+      <visual>
+        <geometry>
+          <box size="0.02 0.02 0.01"/>
+        </geometry>
+        <material name="blue"/>
+      </visual>
+      <inertial>
+        <mass value="0.001"/>
+        <origin xyz="0 0 0" rpy="0 0 0"/>
+        <inertia ixx="1e-6" ixy="0" ixz="0" iyy="1e-6" iyz="0" izz="1e-6"/>
+      </inertial>
+    </link>
+    <joint name="${name}_imu_joint" type="fixed">
+      <parent link="${parent}"/>
+      <child link="${name}_imu_link"/>
+      <origin xyz="0 0 0.0115" rpy="0 0 0"/> <!-- Mounted on top of plate: 1.5mm (half plate) + 10mm (half IMU height) -->
+    </joint>
+    <!--
+      GAZEBO PLUGIN: IMU
+      This plugin makes the IMU sensor publish orientation, angular velocity, and linear acceleration.
+    -->
+    <gazebo reference="${name}_imu_link">
+      <gravity>true</gravity>
+      <sensor name="${name}_imu_sensor" type="imu">
+        <always_on>true</always_on>
+        <update_rate>100</update_rate>
+        <visualize>true</visualize>
+        <topic>__default_topic__</topic>
+        <plugin filename="libgazebo_ros_imu_sensor.so" name="imu_plugin">
+          <topicName>imu</topicName>
+          <bodyName>${name}_imu_link</bodyName>
+          <updateRateHZ>100.0</updateRateHZ>
+          <gaussianNoise>0.0</gaussianNoise>
+          <xyzOffset>0 0 0</xyzOffset>
+          <rpyOffset>0 0 0</rpyOffset>
+          <frameName>${name}_imu_link</frameName>
+          <initialOrientationAsReference>false</initialOrientationAsReference>
+        </plugin>
+        <pose>0 0 0 0 0 0</pose>
+      </sensor>
+    </gazebo>
   </xacro:macro>
 </robot>

Commit message: refactor: Reorganize navigation and SLAM configuration file paths into subdirectories and add explicit color definition for blue material in sensors.xacro.

File: src/sme_robot_mobile_description/urdf/sme_robot_mobile_sensors.xacro (robot description, xacro)
@@ -86,5 +86,7 @@
           <box size="0.02 0.02 0.01"/>
         </geometry>
-        <material name="blue"/>
+        <material name="blue">
+          <color rgba="0 0 1 1"/>
+        </material>
       </visual>
       <inertial>
