Commit message: refactor: Redesign robot base URDF by introducing a virtual chassis and a physical base link, and update RViz configuration to reflect new link structure and add TF display.

File: src/sme_robot_mobile_description/urdf/sme_robot_mobile_base.xacro (robot description, xacro)
@@ -17,38 +17,71 @@
       <parent link="${name}_footprint"/>
       <child link="${name}_chassis"/>
-      <origin xyz="0 0 0.1" rpy="0 0 0"/> <!-- Raise chassis 10cm off ground -->
+      <origin xyz="0 0 0.08" rpy="0 0 0"/> <!-- Raise chassis 8cm off ground (wheel diameter) -->
     </joint>
     <!--
-      CHASSIS LINK
-      The main body of the robot.
+      CHASSIS LINK (Virtual - for collision and inertia)
+      The main body of the robot - invisible, used for physics.
     -->
     <link name="${name}_chassis">
-      <visual>
-        <geometry>
-          <box size="0.5 0.3 0.1"/> <!-- Length 0.5m, Width 0.3m, Height 0.1m -->
-        </geometry>
-        <material name="blue">
-          <color rgba="0 0 0.8 1"/>
-        </material>
-      </visual>
       <collision>
         <geometry>
-          <box size="0.5 0.3 0.1"/>
+          <box size="0.26 0.245 0.12"/>
         </geometry>
+        <material name="black">
+          <color rgba="0.1 0.1 0.1 0.1"/>
+        </material>
       </collision>
       <inertial>
-        <mass value="10.0"/> <!-- Heavy base for stability -->
+        <mass value="15.0"/> <!-- Heavy base for stability -->
         <inertia ixx="0.1" ixy="0" ixz="0" iyy="0.1" iyz="0" izz="0.1"/>
       </inertial>
     </link>
     <!--
+      BOTTOM PLATE
+      Lower acrylic plate (3mm thickness)
+    -->
+    <link name="${name}_base_link">
+      <visual>
+        <geometry>
+          <box size="0.26 0.245 0.003"/> <!-- 26cm x 24.5cm x 3mm -->
+        </geometry>
+        <material name="black">
+          <color rgba="0.1 0.1 0.1 1"/>
+        </material>
+      </visual>
+    </link>
+    <joint name="${name}_base_link_joint" type="fixed">
+      <parent link="${name}_chassis"/>
+      <child link="${name}_base_link"/>
+      <origin xyz="0 0 0" rpy="0 0 0"/> <!-- Bottom of chassis (12cm/2 = 6cm down) -->
+    </joint>
+    <!--
+      TOP PLATE
+      Upper acrylic plate (3mm thickness)
+    -->
+    <link name="${name}_top_plate">
+      <visual>
+        <geometry>
+          <box size="0.26 0.245 0.003"/> <!-- 26cm x 24.5cm x 3mm -->
+        </geometry>
+        <material name="black">
+          <color rgba="0.1 0.1 0.1 1"/>
+        </material>
+      </visual>
+    </link>
+    <joint name="${name}_top_plate_joint" type="fixed">
+      <parent link="${name}_base_link"/>
+      <child link="${name}_top_plate"/>
+      <origin xyz="0 0 0.04" rpy="0 0 0"/> <!-- Top of chassis (12cm/2 = 6cm up) -->
+    </joint>
+    <!--
       WHEEL MACRO
       Helper to create 4 identical wheels.
     -->
-    <xacro:macro name="wheel" params="prefix x_pos y_pos">
-      <link name="${prefix}_wheel">
+    <xacro:macro name="wheel" params="prefix x_pos y_pos z_pos">
+      <link name="${name}_${prefix}_wheel">
         <visual>
           <geometry>
-            <cylinder radius="0.1" length="0.05"/>
+            <cylinder radius="0.04" length="0.037"/> <!-- 80mm diameter, 37mm width -->
           </geometry>
           <material name="black">
@@ -58,5 +91,5 @@
         <collision>
           <geometry>
-            <cylinder radius="0.1" length="0.05"/>
+            <cylinder radius="0.04" length="0.037"/>
           </geometry>
         </collision>
@@ -66,17 +99,20 @@
         </inertial>
       </link>
-      <joint name="${prefix}_wheel_joint" type="continuous">
+      <joint name="${name}_${prefix}_wheel_joint" type="continuous">
         <parent link="${name}_chassis"/>
-        <child link="${prefix}_wheel"/>
+        <child link="${name}_${prefix}_wheel"/>
         <!-- Rotate cylinder to be upright for a wheel -->
-        <origin xyz="${x_pos} ${y_pos} 0" rpy="-1.5707 0 0"/>
+        <origin xyz="${x_pos} ${y_pos} ${z_pos}" rpy="-1.5707 0 0"/>
         <axis xyz="0 0 1"/> <!-- Rotate around the cylinder's Z axis (which is robot's Y) -->
       </joint>
     </xacro:macro>
-    <!-- Instantiate 4 wheels -->
-    <xacro:wheel prefix="front_left"  x_pos="0.2"  y_pos="0.175"/>
-    <xacro:wheel prefix="front_right" x_pos="0.2"  y_pos="-0.175"/>
-    <xacro:wheel prefix="rear_left"   x_pos="-0.2" y_pos="0.175"/>
-    <xacro:wheel prefix="rear_right"  x_pos="-0.2" y_pos="-0.175"/>
+    <!-- Instantiate 4 wheels at corners of 26cm x 24.5cm plate -->
+    <!-- x_pos = 0.26/2 (plate width/2) - 0.04 wheel radius = 0.09 -->
+    <!-- y_pos = 0.245/2 (plate height/2) + 0.0374/2 wheel width = 0.1412 -->
+    <!-- z_pos = -0.04 wheel radius to base link (bottom plate) -->
+    <xacro:wheel prefix="front_left"  x_pos="0.09"  y_pos="0.1412" z_pos="-0.04"/> <!-- robot_base_front_left -->
+    <xacro:wheel prefix="front_right" x_pos="0.09"  y_pos="-0.1412" z_pos="-0.04"/> <!-- robot_base_front_right -->
+    <xacro:wheel prefix="rear_left"   x_pos="-0.09" y_pos="0.1412" z_pos="-0.04"/> <!-- robot_base_rear_left -->
+    <xacro:wheel prefix="rear_right"  x_pos="-0.09" y_pos="-0.1412" z_pos="-0.04"/> <!-- robot_base_rear_right -->
   </xacro:macro>
 </robot>

File: src/sme_robot_mobile_description/urdf/sme_robot_mobile_robot.xacro (robot description, xacro)
@@ -1,4 +1,6 @@
 <?xml version="1.0"?>
-<robot name="robot_description" xmlns:xacro="http://www.ros.org/wiki/xacro">
+<robot name="robot" xmlns:xacro="http://www.ros.org/wiki/xacro">
+  <!-- Define robot name prefix - change this to customize all link/joint names -->
+  <xacro:property name="name" value="robot"/>
   <!-- Include the sub-components -->
   <xacro:include filename="$(find sme_robot_mobile_description)/urdf/sme_robot_mobile_base.xacro"/>
@@ -10,7 +12,7 @@
   -->
   <!-- Create the base with name prefix 'robot' -->
-  <xacro:mobile_base name="robot"/>
-  <!-- Attach sensors to the chassis link -->
-  <xacro:add_sensors parent="robot_chassis"/>
+  <xacro:mobile_base name="${name}"/>
+  <!-- Attach sensors to the top plate -->
+  <xacro:add_sensors name="${name}" parent="${name}_top_plate"/>
   <!--
     GAZEBO PLUGINS
@@ -22,11 +24,11 @@
       <updateRate>100.0</updateRate>
       <robotNamespace>/</robotNamespace>
-      <leftFrontJoint>front_left_wheel_joint</leftFrontJoint>
-      <rightFrontJoint>front_right_wheel_joint</rightFrontJoint>
-      <leftRearJoint>rear_left_wheel_joint</leftRearJoint>
-      <rightRearJoint>rear_right_wheel_joint</rightRearJoint>
-      <wheelSeparation>0.35</wheelSeparation>
-      <wheelDiameter>0.2</wheelDiameter>
-      <robotBaseFrame>robot_footprint</robotBaseFrame>
+      <leftFrontJoint>${name}_front_left_wheel_joint</leftFrontJoint>
+      <rightFrontJoint>${name}_front_right_wheel_joint</rightFrontJoint>
+      <leftRearJoint>${name}_rear_left_wheel_joint</leftRearJoint>
+      <rightRearJoint>${name}_rear_right_wheel_joint</rightRearJoint>
+      <wheelSeparation>0.2824</wheelSeparation> <!-- 2 * 0.1412 (y_pos) -->
+      <wheelDiameter>0.08</wheelDiameter> <!-- 80mm -->
+      <robotBaseFrame>${name}_footprint</robotBaseFrame>
       <torque>20</torque>
       <commandTopic>cmd_vel</commandTopic>

File: src/sme_robot_mobile_description/urdf/sme_robot_mobile_sensors.xacro (robot description, xacro)
@@ -7,10 +7,10 @@
       - parent: The link to attach sensors to.
   -->
-  <xacro:macro name="add_sensors" params="parent">
+  <xacro:macro name="add_sensors" params="name parent">
     <!--
       LIDAR SENSOR
       Used for 2D mapping and navigation (AMCL/Gmapping).
     -->
-    <link name="lidar_link">
+    <link name="${name}_lidar_link">
       <visual>
         <geometry>
@@ -20,8 +20,8 @@
       </visual>
     </link>
-    <joint name="lidar_joint" type="fixed">
+    <joint name="${name}_lidar_joint" type="fixed">
       <parent link="${parent}"/>
-      <child link="lidar_link"/>
-      <origin xyz="0.2 0 0.08" rpy="0 0 0"/> <!-- Mounted on front top of chassis -->
+      <child link="${name}_lidar_link"/>
+      <origin xyz="0 0 0.0265" rpy="0 0 0"/> <!-- Mounted on top of plate: 1.5mm (half plate) + 25mm (half lidar height) -->
     </joint>
     <!--
@@ -29,5 +29,5 @@
       Used for visual perception.
     -->
-    <link name="camera_link">
+    <link name="${name}_camera_link">
       <visual>
         <geometry>
@@ -37,8 +37,8 @@
       </visual>
     </link>
-    <joint name="camera_joint" type="fixed">
+    <joint name="${name}_camera_joint" type="fixed">
       <parent link="${parent}"/>
-      <child link="camera_link"/>
-      <origin xyz="0.25 0 0.05" rpy="0 0 0"/> <!-- Mounted at the very front -->
+      <child link="${name}_camera_link"/>
+      <origin xyz="0.12 0 0.0115" rpy="0 0 0"/> <!-- Mounted on top of plate: 1.5mm (half plate) + 10mm (half camera height) -->
     </joint>
     <!--
@@ -46,6 +46,6 @@
       This plugin makes the lidar sensor actually publish laser scan data in Gazebo.
     -->
-    <gazebo reference="lidar_link">
-      <sensor type="ray" name="lidar_sensor">
+    <gazebo reference="${name}_lidar_link">
+      <sensor type="ray" name="${name}_lidar_sensor">
         <pose>0 0 0 0 0 0</pose>
         <visualize>true</visualize>
@@ -73,5 +73,5 @@
         <plugin name="gazebo_ros_lidar_controller" filename="libgazebo_ros_laser.so">
           <topicName>scan</topicName>
-          <frameName>lidar_link</frameName>
+          <frameName>${name}_lidar_link</frameName>
         </plugin>
       </sensor>

Commit message: updage gazebo classic to gazebo ignition

File: src/sme_robot_mobile_description/urdf/sme_robot_mobile_base.xacro (robot description, xacro)
@@ -21,14 +21,19 @@
     <!--
       CHASSIS LINK (Virtual - for collision and inertia)
-      The main body of the robot - invisible, used for physics.
+      The main body of the robot.
     -->
     <link name="${name}_chassis">
+      <visual>
+        <geometry>
+          <box size="0.26 0.245 0.12"/>
+        </geometry>
+        <material name="black">
+          <color rgba="0.1 0.1 0.1 1"/>
+        </material>
+      </visual>
       <collision>
         <geometry>
           <box size="0.26 0.245 0.12"/>
         </geometry>
-        <material name="black">
-          <color rgba="0.1 0.1 0.1 0.1"/>
-        </material>
       </collision>
       <inertial>
@@ -37,4 +42,13 @@
       </inertial>
     </link>
+    <gazebo reference="${name}_chassis">
+      <visual>
+        <material>
+          <ambient>0.2 0.2 0.2 1</ambient>
+          <diffuse>0.2 0.2 0.2 1</diffuse>
+          <specular>0.2 0.2 0.2 1</specular>
+        </material>
+      </visual>
+    </gazebo>
     <!--
       BOTTOM PLATE
@@ -51,4 +65,13 @@
       </visual>
     </link>
+    <gazebo reference="${name}_base_link">
+      <visual>
+        <material>
+          <ambient>0.1 0.1 0.1 1</ambient>
+          <diffuse>0.1 0.1 0.1 1</diffuse>
+          <specular>0.1 0.1 0.1 1</specular>
+        </material>
+      </visual>
+    </gazebo>
     <joint name="${name}_base_link_joint" type="fixed">
       <parent link="${name}_chassis"/>
@@ -70,4 +93,13 @@
       </visual>
     </link>
+    <gazebo reference="${name}_top_plate">
+      <visual>
+        <material>
+          <ambient>0.1 0.1 0.1 1</ambient>
+          <diffuse>0.1 0.1 0.1 1</diffuse>
+          <specular>0.1 0.1 0.1 1</specular>
+        </material>
+      </visual>
+    </gazebo>
     <joint name="${name}_top_plate_joint" type="fixed">
       <parent link="${name}_base_link"/>
@@ -99,4 +131,13 @@
         </inertial>
       </link>
+      <gazebo reference="${name}_${prefix}_wheel">
+        <visual>
+          <material>
+            <ambient>0.1 0.1 0.1 1</ambient>
+            <diffuse>0.1 0.1 0.1 1</diffuse>
+            <specular>0.1 0.1 0.1 1</specular>
+          </material>
+        </visual>
+      </gazebo>
       <joint name="${name}_${prefix}_wheel_joint" type="continuous">
         <parent link="${name}_chassis"/>

File: src/sme_robot_mobile_description/urdf/sme_robot_mobile_robot.xacro (robot description, xacro)
@@ -20,20 +20,22 @@
   -->
   <gazebo>
-    <!-- Skid Steer Drive Controller (for 4 wheels) -->
-    <plugin name="skid_steer_drive_controller" filename="libgazebo_ros_skid_steer_drive.so">
-      <updateRate>200.0</updateRate> <!-- INCREASED for more stable physics simulation -->
-      <robotNamespace>/</robotNamespace>
-      <leftFrontJoint>${name}_front_left_wheel_joint</leftFrontJoint>
-      <rightFrontJoint>${name}_front_right_wheel_joint</rightFrontJoint>
-      <leftRearJoint>${name}_rear_left_wheel_joint</leftRearJoint>
-      <rightRearJoint>${name}_rear_right_wheel_joint</rightRearJoint>
-      <wheelSeparation>0.2824</wheelSeparation> <!-- 2 * 0.1412 (y_pos) -->
-      <wheelDiameter>0.08</wheelDiameter> <!-- 80mm -->
-      <robotBaseFrame>${name}_footprint</robotBaseFrame>
-      <torque>20</torque>
-      <commandTopic>cmd_vel</commandTopic>
-      <odometryTopic>odom</odometryTopic>
-      <odometryFrame>odom</odometryFrame>
-      <broadcastTF>true</broadcastTF>
+    <!-- Diff Drive (Skid Steer) -->
+    <plugin filename="gz-sim-diff-drive-system" name="gz::sim::systems::DiffDrive">
+      <left_joint>${name}_front_left_wheel_joint</left_joint>
+      <left_joint>${name}_rear_left_wheel_joint</left_joint>
+      <right_joint>${name}_front_right_wheel_joint</right_joint>
+      <right_joint>${name}_rear_right_wheel_joint</right_joint>
+      <wheel_separation>0.2824</wheel_separation>
+      <wheel_radius>0.04</wheel_radius>
+      <odom_publish_frequency>50</odom_publish_frequency>
+      <topic>cmd_vel</topic>
+      <odom_topic>odom</odom_topic>
+      <tf_topic>tf</tf_topic>
+      <frame_id>odom</frame_id>
+      <child_frame_id>${name}_footprint</child_frame_id>
+    </plugin>
+    <!-- Joint State Publisher -->
+    <plugin filename="gz-sim-joint-state-publisher-system" name="gz::sim::systems::JointStatePublisher">
+      <topic>joint_states</topic>
     </plugin>
   </gazebo>

File: src/sme_robot_mobile_description/urdf/sme_robot_mobile_sensors.xacro (robot description, xacro)
@@ -25,4 +25,13 @@
       <origin xyz="0 0 0.0265" rpy="0 0 0"/> <!-- Mounted on top of plate: 1.5mm (half plate) + 25mm (half lidar height) -->
     </joint>
+    <gazebo reference="${name}_lidar_link">
+      <visual>
+        <material>
+          <ambient>0.1 0.1 0.1 1</ambient>
+          <diffuse>0.1 0.1 0.1 1</diffuse>
+          <specular>0.1 0.1 0.1 1</specular>
+        </material>
+      </visual>
+    </gazebo>
     <!--
       CAMERA SENSOR
@@ -37,4 +46,13 @@
       </visual>
     </link>
+    <gazebo reference="${name}_camera_link">
+      <visual>
+        <material>
+          <ambient>0.1 0.1 0.1 1</ambient>
+          <diffuse>0.1 0.1 0.1 1</diffuse>
+          <specular>0.1 0.1 0.1 1</specular>
+        </material>
+      </visual>
+    </gazebo>
     <joint name="${name}_camera_joint" type="fixed">
       <parent link="${parent}"/>
@@ -47,9 +65,10 @@
     -->
     <gazebo reference="${name}_lidar_link">
-      <sensor type="ray" name="${name}_lidar_sensor">
+      <sensor type="gpu_lidar" name="${name}_lidar_sensor">
         <pose>0 0 0 0 0 0</pose>
         <visualize>true</visualize>
         <update_rate>10</update_rate>
-        <ray>
+        <topic>scan</topic>
+        <lidar>
           <scan>
             <horizontal>
@@ -70,9 +89,5 @@
             <stddev>0.01</stddev>
           </noise>
-        </ray>
-        <plugin name="gazebo_ros_lidar_controller" filename="libgazebo_ros_laser.so">
-          <topicName>scan</topicName>
-          <frameName>${name}_lidar_link</frameName>
-        </plugin>
+        </lidar>
       </sensor>
     </gazebo>
@@ -96,4 +111,13 @@
       </inertial>
     </link>
+    <gazebo reference="${name}_imu_link">
+      <visual>
+        <material>
+          <ambient>0.0 0.0 1.0 1</ambient>
+          <diffuse>0.0 0.0 1.0 1</diffuse>
+          <specular>0.1 0.1 0.1 1</specular>
+        </material>
+      </visual>
+    </gazebo>
     <joint name="${name}_imu_joint" type="fixed">
       <parent link="${parent}"/>
@@ -111,15 +135,5 @@
         <update_rate>100</update_rate>
         <visualize>true</visualize>
-        <topic>__default_topic__</topic>
-        <plugin filename="libgazebo_ros_imu_sensor.so" name="imu_plugin">
-          <topicName>imu</topicName>
-          <bodyName>${name}_imu_link</bodyName>
-          <updateRateHZ>50.0</updateRateHZ>
-          <gaussianNoise>0.0</gaussianNoise>
-          <xyzOffset>0 0 0</xyzOffset>
-          <rpyOffset>0 0 0</rpyOffset>
-          <frameName>${name}_imu_link</frameName>
-          <initialOrientationAsReference>false</initialOrientationAsReference>
-        </plugin>
+        <topic>imu</topic>
         <pose>0 0 0 0 0 0</pose>
       </sensor>
